File: Contra.kicad_pcb (KiCad board)
At the start: 2 copper layers, 231 x 76.2 mm, 110 parts, among them J1 Conn_01x04, SW1 SW_PUSH, U1 ProMicro

Commit message: Modified pcb
Parts:
- removed the G*** at (178.4, 64.1)
- removed the G*** at (119.9, 66.7)
- removed the G*** at (228.6, 65.1) (x2)
- removed the G*** at (253.2, 100.0)
- added G***: LOGO, homerow:homerow_small, B.Cu at (193.0, 66.0)
Other:
- net class Default removed
- net class Power removed
- board text added: "Contra PCB Rev 2.0"
- board text removed: "Contra PCB by ai03 Revision 2.0"
